Commit message: feat(config): add 'setup' named target (initial raised pose)
Add a 'setup' group_state to arm_moveit_config matching the arm's initial
powered-on rest pose (shoulder_lift 1.83, elbow_flex 1.78). To make it
reachable by the planner:

- Widen shoulder_lift upper limit 1.7453->1.9199 and elbow_flex
  1.69->1.85 in dt_arm_moveit_config URDF (the xacro move_group actually
  loads) and mirror in dt_arm_description URDF. The real arm reaches this
  range under torque, so the previous soft limits were too tight.
- Disable self-collision for shoulder_link<->lower_arm_link and
  upper_arm_link<->wrist_link: the folded setup pose flags these as
  contacts in the (conservative) collision model, but the real arm rests
  there collision-free.

Verified: /check_state_validity reports valid (0 contacts) and plan_only
to 'setup' returns SUCCESS.

Co-Authored-By: Claude Opus 4.8 (1M context) <noreply@anthropic.com>

File: src/dt_arm_description/urdf/soarm101_40mmUP.urdf (robot description, URDF)
Before this commit: robot soarm101_40mmUP, 7 links, 6 joints
Joints:
- joint elbow_flex: limit lower=-1.69 upper=1.69 effort=10 velocity=10 -> lower=-1.69 upper=1.85 effort=10 velocity=10
- joint shoulder_lift: limit lower=-1.7453 upper=1.7453 effort=10 velocity=10 -> lower=-1.7453 upper=1.9199 effort=10 velocity=10
